File: Design/AFE - Top level.kicad_sch (KiCad schematic)
At the start: 1 part, among them U3 MC33774ASA1AE-IOs

Commit message: new frame work for the design
Parts:
- removed U3: MC33774ASA1AE-IOs, MC33774ASP1AE_AFE:QFP50P1200X1200X160-65N, symbol MC33774ASA1AE:MC33774ASA1AE
- added U1: MC33774ASA1AE-IOs, MC33774ASP1AE_AFE:QFP50P1200X1200X160-65N, symbol MC33774ASA1AE:MC33774ASA1AE
Connections:
- no-connect marks 0 -> 8
Other:
- added sheet AFE - Cell Balancing (AFE - Cell Balancing.kicad_sch)
- added sheet AFE - Cell_Input (AFE - Cell_Input.kicad_sch)
Changed lines of the file:
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@@
 		(rev "1.0.0")
 	)
+	(no_connect
+		(at 128.27 119.38)
+	)
+	(no_connect
+		(at 128.27 114.3)
+	)
+	(no_connect
+		(at 128.27 124.46)
+	)
+	(no_connect
+		(at 128.27 106.68)
+	)
+	(no_connect
+		(at 128.27 116.84)
+	)
+	(no_connect
+		(at 128.27 109.22)
+	)
+	(no_connect
+		(at 128.27 111.76)
+	)
+	(no_connect
+		(at 128.27 121.92)
+	)
 	(bus_entry
 		(at 119.38 67.31)
@@
 	(bus
 		(pts
-			(xy 167.64 55.88) (xy 173.99 55.88)
+			(xy 167.64 55.88) (xy 189.23 55.88)
 		)
 		(stroke
@@
 	(bus
 		(pts
-			(xy 111.76 57.15) (xy 119.38 57.15)
-		)
-		(stroke
-			(width 0)
-			(type default)
-		)
-	)
-	(bus
-		(pts
 			(xy 119.38 64.77) (xy 119.38 62.23)
 		)
@@
 		(pts
 			(xy 156.21 69.85) (xy 165.1 69.85)
+		)
+		(stroke
+			(width 0)
+			(type default)
+		)
+	)
+	(bus
+		(pts
+			(xy 92.71 57.15) (xy 119.38 57.15)
 		)
 		(stroke
@@
 	(text "[${#}] ${SHEETNAME}"
 		(exclude_from_sim no)
-		(at 145.542 22.86 0)
+		(at 144.018 18.034 0)
 		(effects
 			(font
 				(face "Times New Roman")
-				(size 8 8)
+				(size 6 6)
 				(thickness 1.6)
 				(bold yes)
@@
 		)
 	)
-	(hierarchical_label "CT[0..18]"
-		(shape input)
-		(at 111.76 57.15 180)
+	(label "CT[0..18]"
+		(at 101.6 57.15 0)
 		(fields_autoplaced yes)
 		(effects
 			(font
+				(face "Arial")
 				(size 1.27 1.27)
-			)
-			(justify right)
-		)
-	)
-	(hierarchical_label "CB[0..18]"
-		(shape input)
+				(thickness 0.254)
+				(bold yes)
+			)
+			(justify left bottom)
+		)
+	)
+	(label "CB[0..18]"
 		(at 173.99 55.88 0)
 		(fields_autoplaced yes)
 		(effects
 			(font
+				(face "Arial")
 				(size 1.27 1.27)
-			)
-			(justify left)
+				(thickness 0.254)
+				(bold yes)
+			)
+			(justify left bottom)
 		)
 	)
 	(symbol
+		(lib_name "MC33774ASA1AE_1")
 		(lib_id "MC33774ASA1AE:MC33774ASA1AE")
 		(at 143.51 91.44 0)
@@
 		(dnp no)
 		(fields_autoplaced yes)
-		(property "Reference" "U3"
+		(property "Reference" "U1"
 			(at 142.24 46.99 0)
 			(effects
@@
 		)
 		(property "Footprint" "MC33774ASP1AE_AFE:QFP50P1200X1200X160-65N"
-			(at 154.178 127 0)
+			(at 154.686 139.192 0)
 			(effects
 				(font
@@
 		)
 		(property "Description" "18 Ch AFE"
-			(at 161.29 122.936 0)
+			(at 160.02 134.62 0)
 			(effects
 				(font
@@
 			)
 		)
+		(pin "48"
+		)
+		(pin "55"
+		)
+		(pin "3"
+		)
+		(pin "28"
+		)
+		(pin "20"
+		)
+		(pin "52"
+		)
+		(pin "5"
+		)
+		(pin "39"
+		)
+		(pin "7"
+		)
+		(pin "36"
+		)
+		(pin "23"
+		)
+		(pin "9"
+		)
+		(pin "13"
+		)
+		(pin "47"
+		)
+		(pin "38"
+		)
+		(pin "6"
+		)
+		(pin "11"
+		)
+		(pin "12"
+		)
+		(pin "18"
+		)
+		(pin "33"
+		)
+		(pin "34"
+		)
+		(pin "40"
+		)
+		(pin "26"
+		)
+		(pin "31"
+		)
+		(pin "57"
+		)
+		(pin "27"
+		)
+		(pin "4"
+		)
+		(pin "58"
+		)
+		(pin "15"
+		)
+		(pin "49"
+		)
+		(pin "30"
+		)
+		(pin "14"
+		)
+		(pin "16"
+		)
+		(pin "50"
+		)
+		(pin "46"
+		)
+		(pin "51"
+		)
+		(pin "53"
+		)
+		(pin "56"
+		)
+		(pin "25"
+		)
+		(pin "19"
+		)
+		(pin "10"
+		)
+		(pin "24"
+		)
+		(pin "35"
+		)
+		(pin "8"
+		)
+		(pin "17"
+		)
 		(pin "22"
 		)
-		(pin "51"
-		)
-		(pin "25"
-		)
-		(pin "17"
-		)
 		(pin "2"
 		)
-		(pin "23"
-		)
-		(pin "26"
+		(pin "54"
+		)
+		(pin "29"
+		)
+		(pin "32"
 		)
 		(pin "37"
 		)
-		(pin "52"
-		)
-		(pin "53"
-		)
-		(pin "29"
-		)
-		(pin "10"
-		)
-		(pin "27"
-		)
-		(pin "36"
-		)
-		(pin "57"
-		)
-		(pin "14"
-		)
-		(pin "31"
-		)
-		(pin "32"
-		)
-		(pin "18"
-		)
-		(pin "3"
-		)
-		(pin "39"
-		)
-		(pin "5"
-		)
-		(pin "11"
-		)
-		(pin "16"
-		)
-		(pin "20"
-		)
-		(pin "38"
-		)
-		(pin "4"
-		)
-		(pin "40"
-		)
-		(pin "33"
-		)
-		(pin "55"
-		)
-		(pin "28"
-		)
-		(pin "24"
-		)
-		(pin "56"
-		)
-		(pin "58"
-		)
-		(pin "6"
-		)
-		(pin "35"
-		)
-		(pin "13"
-		)
-		(pin "54"
-		)
-		(pin "7"
-		)
-		(pin "8"
-		)
-		(pin "9"
-		)
-		(pin "19"
-		)
-		(pin "15"
-		)
-		(pin "12"
-		)
-		(pin "30"
-		)
-		(pin "34"
-		)
 		(instances
-			(project ""
+			(project "BMS_Design"
 				(path "/d3cbbc2c-48ef-45dd-b1b3-b57e1b62c15c/a6f6d1e1-9a1e-4a49-9157-1184d73c923a/3ba4dcbb-6b17-48b1-9055-15badbca1f49"
-					(reference "U3")
+					(reference "U1")
 					(unit 1)
 				)
 			)
+		)
+	)
+	(sheet
+		(at 189.23 53.34)
+		(size 26.67 53.34)
+		(fields_autoplaced yes)
+		(stroke
+			(width 0.25)
+			(type solid)
+			(color 255 129 18 1)
+		)
+		(fill
+			(color 255 129 18 0.5000)
+		)
+		(property "Sheetname" "AFE - Cell Balancing"
+			(at 189.23 52.2146 0)
+			(effects
+				(font
+					(face "Arial")
+					(size 2 2)
+					(thickness 0.4)
+					(bold yes)
+				)
+				(justify left bottom)
+			)
+		)
+		(property "Sheetfile" "AFE - Cell Balancing.kicad_sch"
+			(at 189.23 107.3134 0)
+			(effects
+				(font
+					(size 1.27 1.27)
+				)
+				(justify left top)
+				(hide yes)
+			)
+		)
+		(pin "CB[0..18]" output
+			(at 189.23 55.88 180)
+			(effects
+				(font
+					(size 1.27 1.27)
+				)
+				(justify left)
+			)
+		)
+		(instances
+			(project "BMS_Design"
+				(path "/d3cbbc2c-48ef-45dd-b1b3-b57e1b62c15c/a6f6d1e1-9a1e-4a49-9157-1184d73c923a/3ba4dcbb-6b17-48b1-9055-15badbca1f49"
+					(page "11")
+				)
+			)
+		)
+	)
+	(sheet
+		(at 69.85 54.61)
+		(size 22.86 66.04)
+		(fields_autoplaced yes)
+		(stroke
+			(width 0.25)
+			(type solid)
+			(color 255 248 60 1)
+		)
+		(fill
+			(color 255 248 60 0.5100)
+		)
+		(property "Sheetname" "AFE - Cell_Input"
+			(at 69.85 53.4846 0)
+			(effects
+				(font
+					(face "Arial")
+					(size 2 2)
+					(thickness 0.4)
+					(bold yes)
+				)
+				(justify left bottom)
+			)
+		)
+		(property "Sheetfile" "AFE - Cell_Input.kicad_sch"
+			(at 69.85 121.2834 0)
+			(effects
+				(font
+					(size 1.27 1.27)
+				)
+				(justify left top)
+				(hide yes)
+			)
+		)
+		(pin "CT[0..18]" output
+			(at 92.71 57.15 0)
+			(effects
+				(font
+					(size 1.27 1.27)
+				)
+				(justify right)
+			)
+		)
+		(instances
+			(project "BMS_Design"
+				(path "/d3cbbc2c-48ef-45dd-b1b3-b57e1b62c15c/a6f6d1e1-9a1e-4a49-9157-1184d73c923a/3ba4dcbb-6b17-48b1-9055-15badbca1f49"
+					(page "10")
+				)
+			)
