File: Design/BMS_Design.kicad_sch (KiCad schematic)
At the start: 0 parts

Commit message: created base model
Other:
- removed sheet AFE
- removed sheet Chg_disChg_MOSFET
- removed sheet MCU
- added sheet Project_Architecture (Project_Architecture.kicad_sch)
- note added: "${BOARD_NAME}"
- note added: "..........................................."
- note added: "Bottom Side"
- note added: "Cover Page"
- note added: "DATE : {DATE}"
- note added: "Designer : {NAME}"
- note added: "Index"
- note added: "MCU"
- note added: "Power - Sequencing"
- note added: "Project Architecture"
- note added: "REV : {REV}"
- note added: "Random Sheet 1"
- note added: "Random Sheet 2"
- note added: "Revision History"
- note added: "Top Side"

Commit message: new frame work for the design
Other:
- added sheet Block_Diagram (Block_Diagram.kicad_sch)
- note added: "AFE - Cell_Balancing"
- note added: "AFE - Cell_Input"
- note added: "AFE - Top Level"
- note added: "Block_Diagram"
- note added: "CHG_DCHG - MOSFET"
- note added: "CHG_DCHG - Top level"
- note added: "Comm - CAN"
- note added: "Comm - RS-485"
- note added: "DATE : ${DATE}"
- note added: "Designer : ${NAME}"
- note added: "Indication - PWR"
- note added: "Indication - USR"
- note added: "Interface - Interconnects"
- note added: "MCU - IO"
- note added: "Misc - Holes,Fid"
- note added: "Power - Connectors"
- note added: "Power - Generation"
- note added: "Power - MCU,AFE"
- note added: "Pre - charge_Circuit"
- note added: "Project_Architecture"
- note added: "Protection - Fuse"
- note added: "REV : ${REV}"
- note added: "Sensing - Current"
- note added: "Sensing - Hum_Press"
- note added: "Sensing - Temp"
- note removed: "..........................................."
- note removed: "Cover Page"
- note removed: "DATE : {DATE}"
- note removed: "Designer : {NAME}"
- note removed: "MCU"
- note removed: "Power - Sequencing"
- note removed: "Project Architecture"
- note removed: "REV : {REV}"
- note removed: "Random Sheet 1"
- note removed: "Random Sheet 2"
- note removed: "Revision History"
