File: Design/MCU_AFE_Power.kicad_sch (KiCad schematic)
At the start: 0 parts

Commit message: new frame work for the design
Parts:
- added U2: MC33774ASA1AE-IOs, MC33774ASP1AE_AFE:QFP50P1200X1200X160-65N, symbol MC33774ASA1AE:MC33774ASA1AE
Other:
- note added: "[${#}] ${SHEETNAME}"
