File: Design/MOSFET_CHG_DCHG.kicad_sch (KiCad schematic)
At the start: 0 parts

Commit message: new frame work for the design
Other:
- added sheet CHG_DCHG - MOSFET (CHG_DCHG - MOSFET.kicad_sch)
- added sheet Pre-charge_Circuit (Pre-charge_Circuit.kicad_sch)
- note added: "[${#}] ${SHEETNAME}"
Changed lines of the file:
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@@
 	(title_block
 		(title "Cell_Sentinel")
-		(date "2024-09-03")
+		(date "2024-11-05")
 		(rev "1.0.0")
 	)
+	(text "[${#}] ${SHEETNAME}"
+		(exclude_from_sim no)
+		(at 139.954 19.558 0)
+		(effects
+			(font
+				(face "Times New Roman")
+				(size 6 6)
+				(thickness 1.6)
+				(bold yes)
+				(color 159 72 15 1)
+			)
+		)
+	)
+	(sheet
+		(at 149.86 52.07)
+		(size 35.56 99.06)
+		(stroke
+			(width 0.25)
+			(type solid)
+			(color 241 93 255 1)
+		)
+		(fill
+			(color 241 93 255 0.5000)
+		)
+		(property "Sheetname" "CHG_DCHG - MOSFET"
+			(at 149.86 51.054 0)
+			(effects
+				(font
+					(face "Arial")
+					(size 2 2)
+					(thickness 0.254)
+					(bold yes)
+				)
+				(justify left bottom)
+			)
+		)
+		(property "Sheetfile" "CHG_DCHG - MOSFET.kicad_sch"
+			(at 149.86 65.3546 0)
+			(effects
+				(font
+					(size 1.27 1.27)
+				)
+				(justify left top)
+				(hide yes)
+			)
+		)
+		(instances
+			(project "BMS_Design"
+				(path "/d3cbbc2c-48ef-45dd-b1b3-b57e1b62c15c/a6f6d1e1-9a1e-4a49-9157-1184d73c923a/e9678301-b11c-4ec8-96b9-98915a57482b"
+					(page "14")
+				)
+			)
+		)
+	)
+	(sheet
+		(at 63.5 50.8)
+		(size 31.75 104.14)
+		(stroke
+			(width 0.25)
+			(type solid)
+			(color 137 72 255 1)
+		)
+		(fill
+			(color 1 0 255 0.5020)
+		)
+		(property "Sheetname" "Pre-charge_Circuit"
+			(at 63.5 49.784 0)
+			(effects
+				(font
+					(face "Arial")
+					(size 2 2)
+					(thickness 0.254)
+					(bold yes)
+				)
+				(justify left bottom)
+			)
+		)
+		(property "Sheetfile" "Pre-charge_Circuit.kicad_sch"
+			(at 63.5 64.0846 0)
+			(effects
+				(font
+					(size 1.27 1.27)
+				)
+				(justify left top)
+				(hide yes)
+			)
+		)
+		(instances
+			(project "BMS_Design"
+				(path "/d3cbbc2c-48ef-45dd-b1b3-b57e1b62c15c/a6f6d1e1-9a1e-4a49-9157-1184d73c923a/e9678301-b11c-4ec8-96b9-98915a57482b"
+					(page "13")
+				)
+			)
+		)
+	)
 )
