File: Design/Pre-charge_Circuit.kicad_sch (KiCad schematic)
At the start: 0 parts

Commit message: new frame work for the design
Other:
- note added: "[${#}] ${SHEETNAME}"
Changed lines of the file:
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@@
 	(title_block
 		(title "Cell_Sentinel")
-		(date "2024-09-03")
+		(date "2024-11-05")
 		(rev "1.0.0")
 	)
+	(text "[${#}] ${SHEETNAME}"
+		(exclude_from_sim no)
+		(at 137.668 17.78 0)
+		(effects
+			(font
+				(face "Times New Roman")
+				(size 6 6)
+				(thickness 1.6)
+				(bold yes)
+				(color 159 72 15 1)
+			)
+		)
+	)
 )
