File: Design/Project_Architecture.kicad_sch (KiCad schematic)
At the start: 0 parts

Commit message: new frame work for the design
Other:
- sheet AFE renamed AFE - Top level
- sheet Communication renamed Comm - RS-485
- sheet Current_Sense renamed Sensing - Current
- sheet MCU - IOs renamed MCU - IO
- sheet MCU_AFE_Power renamed Power - MCU,AFE
- sheet Power_Conversion renamed Power - Generation
- sheet Protection_Circuits renamed Protection - Fuse
- removed sheet CELL
- removed sheet MOSFET_CHG_DCHG
- removed sheet Pre-charge_Circuit
- added sheet CHG_DCHG -Top_level (MOSFET_CHG_DCHG.kicad_sch)
- added sheet Comm - CAN (Comm - CAN.kicad_sch)
- added sheet Indication - PWR (Indication - PWR.kicad_sch)
- added sheet Indication - USR (Indication - USR.kicad_sch)
- added sheet Interface - Interconnects (Interface - Interconnects.kicad_sch)
- added sheet Misc - Holes,Fid (Misc - Holes,Fid.kicad_sch)
- added sheet Power - Connectors (Power - Connectors.kicad_sch)
- added sheet Sensing - Hum_Press (Sensing - Hum_Press.kicad_sch)
- added sheet Sensing - Temp (Sensing - Temp.kicad_sch)
- sheet AFE - Top level: file AFE.kicad_sch -> AFE - Top level.kicad_sch
- sheet Comm - RS-485: file Communication.kicad_sch -> Comm - RS-485.kicad_sch
- sheet MCU - IO: file MCU.kicad_sch -> MCU - IO.kicad_sch
- sheet Power - Generation: file Power_Conversion.kicad_sch -> Power - Generation.kicad_sch
- sheet Power - MCU,AFE: file MCU_AFE_Power.kicad_sch -> Power - MCU,AFE.kicad_sch
- sheet Protection - Fuse: file Protection_Circuits.kicad_sch -> Protection - Fuse.kicad_sch
- sheet Sensing - Current: file Current_Sense.kicad_sch -> Sensing - Current.kicad_sch
- note added: "[${#}] ${SHEETNAME}"
